File: HW/TRX_MODULE/TRX_MODULE/TRX_MODULE.kicad_pcb (KiCad board)
At the start: 2 copper layers, 100 x 100 mm, 42 parts, among them J1 Conn_Coaxial, J2 Conn_Coaxial, J4 HEADER_2x26, J5 JTAG, M1 HOLE, M2 HOLE, M3 HOLE, M4 HOLE, Q1 BC817, U1 E19-433M30S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

Commit message: update
Parts:
- added C24: 100nF, Capacitors_SMD:C_0603, F.Cu at (-25.4, -64.8)
- added C25: 100nF, Capacitors_SMD:C_0603, F.Cu at (-20.8, -70.5)
- added C26: 10uF, Capacitors_SMD:C_0603, F.Cu at (-17.4, -70.5)
- added CON5: JTAG, Mlab_Pin_Headers:Straight_2x07, F.Cu at (-19.0, 36.0)
- added J1: 0, Resistors_THT:R_Axial_DIN0204_L3.6mm_D1.6mm_P1.90mm_Vertical, F.Cu at (-34.8, -24.1)
- added J2: 0, Resistors_THT:R_Axial_DIN0204_L3.6mm_D1.6mm_P1.90mm_Vertical, F.Cu at (-34.8, -21.6)
- added J3: 0, Resistors_THT:R_Axial_DIN0204_L3.6mm_D1.6mm_P1.90mm_Vertical, F.Cu at (-34.8, -19.1)
- added J4: 0, Resistors_THT:R_Axial_DIN0204_L3.6mm_D1.6mm_P1.90mm_Vertical, F.Cu at (-34.8, -16.5)
- added R1: 10k, Resistors_SMD:R_0603, F.Cu at (-19.0, 40.2)
- added R10: 10k, Resistors_SMD:R_0603, F.Cu at (-27.6, 19.3)
- added R2: 10k, Resistors_SMD:R_0603, F.Cu at (-11.4, 31.8)
- added R3: 10k, Resistors_SMD:R_0603, F.Cu at (-16.4, 40.2)
- added R4: 10k, Resistors_SMD:R_0603, F.Cu at (-59.4, 12.2)
- added R8: 10k, Resistors_SMD:R_0603, F.Cu at (-27.6, 16.1)
- added R9: 10k, Resistors_SMD:R_0603, F.Cu at (-27.6, 17.7)
- C5: value ? -> 100nF
- J5: value JTAG -> 0; footprint Mlab_Pin_Headers:Straight_2x07 -> Resistors_THT:R_Axial_DIN0204_L3.6mm_D1.6mm_P1.90mm_Vertical
- moved C4 107.0 mm to (-13.9, 40.3), turned to 270 degrees
- moved C3 99.4 mm to (-11.7, 40.5), turned to 270 degrees
- moved C23 64.5 mm to (-35.3, -6.35), turned to 180 degrees
- moved C22 60.1 mm to (-15.7, -6.86), turned to 180 degrees
- moved U3 42.1 mm to (-18.1, 22.1)
- moved X1 42.1 mm to (-20.7, 12.9)
- moved Q1 41.5 mm to (-26.6, 23.9)
- moved D1 39.2 mm to (-10.7, 7.70), turned to 0 degrees
- moved R7 31.1 mm to (-32.8, -8.13), turned to 90 degrees
- moved R6 25.6 mm to (-30.0, -6.35), turned to 180 degrees
- moved R5 23.8 mm to (-32.8, -4.57), turned to 90 degrees
- moved J5 21.0 mm to (-34.8, -13.9), turned to 0 degrees
- moved D4 20.6 mm to (-31.8, 17.7)
- moved U4 18.6 mm to (-23.4, -6.35), turned to 180 degrees
- moved D3 15.9 mm to (-31.8, 19.6)
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- renumbered J1 to CON1, J2 to CON2, J4 to CON4
Connections:
- net reset renamed RESET
- CON4 pad 1: +5V -> +12V_A
- CON4 pad 10: +1V2 -> +5V_B
- CON4 pad 11: GND -> +5V_C
- CON4 pad 12: GND -> +5V_C
- CON4 pad 13: (no net) -> +5V_D
- CON4 pad 14: CAN_H -> +5V_D
- CON4 pad 15: GND -> +5V_E
- CON4 pad 16: GND -> +5V_E
- CON4 pad 17: (no net) -> GND
- CON4 pad 18: CAN_L -> GND
- CON4 pad 2: +5V -> +12V_A
- CON4 pad 20: (no net) -> CAN_L
- CON4 pad 21: (no net) -> GND
- CON4 pad 22: (no net) -> GND
- CON4 pad 24: (no net) -> CAN_H
- CON4 pad 3: GND -> +12V_B
- CON4 pad 4: GND -> +12V_B
- CON4 pad 5: +3V3 -> GND
- CON4 pad 52: (no net) -> 1PPS
- CON4 pad 6: +3V3 -> GND
- CON4 pad 7: GND -> +5V_A
- CON4 pad 8: GND -> +5V_A
- CON4 pad 9: +1V2 -> +5V_B
- D2 pad 2: (no net) -> Net-(D2-Pad2)
- D3 pad 2: (no net) -> Net-(D3-Pad2)
- D4 pad 2: (no net) -> Net-(D4-Pad2)
- J5 pad 1: TDI -> +5V_E
- J5 pad 2: GND -> +5V
- U3 pad 17: (no net) -> Net-(R8-Pad2)
- U3 pad 18: (no net) -> Net-(R9-Pad2)
- U3 pad 19: (no net) -> Net-(R10-Pad2)
- U3 pad 8: (no net) -> 1PPS
Routing:
- net /MOSI_1: track 0.00 -> 68.2 mm, vias 0 -> 2
- net /MISO_1: track 0.00 -> 64.1 mm, vias 0 -> 2
- net /SCK_1: track 0.00 -> 61.1 mm, vias 0 -> 2
- net /TXEN_1: track 0.00 -> 47.3 mm
- net /RXEN_2: track 0.00 -> 44.7 mm
- net /SCK_0: track 0.00 -> 17.0 mm
- net /CS_0: track 0.00 -> 17.0 mm
- net /MISO_0: track 0.00 -> 17.0 mm, vias 0 -> 2
- net /MOSI_0: track 0.00 -> 17.0 mm
- net TDO: track 0.00 -> 16.5 mm
- net CAN_H: track 0.00 -> 13.6 mm
- net CAN_L: track 0.00 -> 13.6 mm
- net TDI: track 0.00 -> 12.5 mm
- net TCKOUT: track 0.00 -> 12.0 mm
- net TMS: track 0.00 -> 10.7 mm, vias 0 -> 1
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Other:
- outline, holes or cut-outs redrawn

Commit message: update
Parts:
- C12, C13, C14, C15, C16, C6, C7, C8, C9: value ? -> 100nF; moved to B.Cu
- moved C8 75.1 mm to (-16.7, 4.62), turned to 90 degrees
- moved C14 73.7 mm to (-22.4, 3.60)
- moved C13 70.2 mm to (-22.4, 1.62)
- moved C12 68.7 mm to (-17.6, -4.92), turned to 270 degrees
- moved C15 66.3 mm to (-18.1, 4.62), turned to 90 degrees
- moved C6 62.3 mm to (-21.2, -4.95), turned to 270 degrees
- moved C16 61.8 mm to (-12.6, 0.53), turned to 180 degrees
- moved C7 56.3 mm to (-12.6, -0.93), turned to 180 degrees
- moved C9 55.4 mm to (-16.2, -4.95), turned to 270 degrees
- moved C22 30.5 mm to (-16.1, 23.6)
- moved C23 30.5 mm to (-35.7, 24.1)
- moved R6 30.5 mm to (-30.3, 24.1)
- moved R7 30.5 mm to (-33.1, 22.3)
- moved U4 30.5 mm to (-23.7, 24.1)
- moved R5 30.5 mm to (-33.1, 25.9)
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Connections:
- CON4 pad 20: CAN_L -> (no net)
- CON4 pad 24: CAN_H -> (no net)
- CON4 pad 44: (no net) -> CAN_L
- CON4 pad 45: (no net) -> GND
- CON4 pad 46: (no net) -> GND
- CON4 pad 48: (no net) -> CAN_H
- CON4 pad 49: (no net) -> GND
- CON4 pad 50: (no net) -> GND
Routing:
- net /TXEN_2: track 0.00 -> 61.4 mm
- net /RXEN_1: track 0.00 -> 38.2 mm
- net +3V3: track 0.00 -> 24.9 mm, vias 0 -> 6
- net /TXEN_1: track 47.3 -> 34.4 mm
- net /RXEN_2: track 44.7 -> 57.3 mm
- net +1V2: track 0.00 -> 8.32 mm, vias 0 -> 3
- net /MOSI_1: track 68.2 -> 63.0 mm, vias 2 -> 3
- net /MISO_1: track 64.1 -> 60.4 mm, vias 2 -> 3
- net /SCK_1: track 61.1 -> 58.0 mm, vias 2 -> 3
- net Net-(Q1-Pad1): track 0.00 -> 2.80 mm
- net Net-(U3-Pad12): track 2.36 -> 2.90 mm

Commit message: update
Routing:
- net /TXEN_1: track 34.4 -> 35.3 mm
Changed lines of the file:
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@@
-(kicad_pcb (version 20171130) (host pcbnew "(5.0-dev-4082-g0504a6d)")
+(kicad_pcb (version 20171130) (host pcbnew "(5.0.0-rc2-dev-411-g5ef715f3d)")
   (general
     (thickness 1.6)
@@
   (segment (start -23.125 3.075) (end -23.839998 3.075) (width 0.3) (layer F.Cu) (net 15))
   (segment (start -23.839998 3.075) (end -24.389998 2.525) (width 0.3) (layer F.Cu) (net 15))
-  (segment (start 16.24 -8.238) (end 16.24 -7.5) (width 0.3) (layer F.Cu) (net 20))
-  (segment (start 13.678 -10.8) (end 16.24 -8.238) (width 0.3) (layer F.Cu) (net 20))
-  (segment (start 0.5 -10.8) (end 13.678 -10.8) (width 0.3) (layer F.Cu) (net 20))
-  (segment (start -0.674989 -9.625011) (end 0.5 -10.8) (width 0.3) (layer F.Cu) (net 20))
-  (segment (start -0.674989 -6.992889) (end -0.674989 -9.625011) (width 0.3) (layer F.Cu) (net 20))
-  (segment (start -11.725 -3.425) (end -4.242878 -3.425) (width 0.3) (layer F.Cu) (net 20))
-  (segment (start -4.242878 -3.425) (end -0.674989 -6.992889) (width 0.3) (layer F.Cu) (net 20))
   (segment (start 17.4 -11.35) (end 18.78 -9.97) (width 0.3) (layer F.Cu) (net 21))
   (segment (start 18.78 -9.97) (end 18.78 -7.5) (width 0.3) (layer F.Cu) (net 21))
@@
   (segment (start -15.675 -8.475) (end -15.675 -5.875) (width 0.25) (layer F.Cu) (net 19))
   (segment (start -15.190126 -15.050335) (end -15.239626 -15.039036) (width 0.25) (layer F.Cu) (net 19))
+  (segment (start 16.24 -9.76) (end 16.24 -7.5) (width 0.3) (layer F.Cu) (net 20))
+  (segment (start -4.242878 -3.425) (end -0.674989 -6.992889) (width 0.3) (layer F.Cu) (net 20))
+  (segment (start -11.725 -3.425) (end -4.242878 -3.425) (width 0.3) (layer F.Cu) (net 20))
+  (segment (start -0.674989 -6.992889) (end -0.674989 -9.625011) (width 0.3) (layer F.Cu) (net 20))
+  (segment (start -0.674989 -9.625011) (end 0.5 -10.8) (width 0.3) (layer F.Cu) (net 20))
+  (segment (start 0.5 -10.8) (end 15.2 -10.8) (width 0.3) (layer F.Cu) (net 20))
+  (segment (start 15.2 -10.8) (end 16.24 -9.76) (width 0.3) (layer F.Cu) (net 20))
   (segment (start -36.272 26.853) (end -33.116 26.853) (width 0.6) (layer F.Cu) (net 26))
   (segment (start -36.46 26.665) (end -36.272 26.853) (width 0.6) (layer F.Cu) (net 26))

Commit message: update
Parts:
- moved C5 43.3 mm to (-5.40, -17.2), turned to 90 degrees
Routing:
- net RESET: track 0.00 -> 38.9 mm, vias 0 -> 1
- net /CAN_RX: track 0.00 -> 27.9 mm
- net /CAN_TX: track 0.00 -> 25.0 mm
- net Net-(CON5-Pad7): track 0.00 -> 2.18 mm
- net +1V2: track 8.32 -> 9.61 mm, vias 3 -> 4
