File: HW/TRX_MODULE/TRX_MODULE/TRX_MODULE.sch (KiCad schematic (older format))
At the start: 51 parts, among them J1 Conn_Coaxial, J2 Conn_Coaxial, J4 HEADER_2x26, J5 JTAG, M1 HOLE, M2 HOLE, M3 HOLE, M4 HOLE, Q1 BC817, U1 E19-433M30S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

Commit message: update
Parts:
- added C24, C25: 100nF, Capacitors_SMD:C_0603, symbol device:C_Small
- added C26: 10uF, Capacitors_SMD:C_0603, symbol device:C_Small
- added J1, J2, J3, J4, J5: 0, Resistors_THT:R_Axial_DIN0204_L3.6mm_D1.6mm_P1.90mm_Vertical, symbol device:R
- added R11: 510, symbol device:R
- added R12: 300, symbol device:R
- added U5: LM1117-3.3, symbol regul:LM1117-3.3
- C5: value ? -> 100nF
- R1, R10, R2, R3, R4, R8, R9: footprint (none) -> Resistors_SMD:R_0603
- renumbered J1 to CON1, J2 to CON2, J4 to CON4, J5 to CON5
Connections:
- net +1V2: now also R11.1, R12.2; no longer CON4.10, CON4.9
- net +3V3: now also C25.2, C26.2, R11.2, U5.2 (VO); no longer CON4.5, CON4.6
- net +5V: now also C24.1, J1.2, J2.2, J3.2, J4.2, J5.2, U5.3 (VI); no longer CON4.1, CON4.2
- net CAN_H: now also CON4.24; no longer CON4.14
- net CAN_L: now also CON4.20; no longer CON4.18
- net GND: now also CON4.17, CON4.18, CON4.21, CON4.22, CON4.5, CON4.6, C24.2, C25.1, C26.1, R12.1, U5.1 (GND); no longer CON4.11, CON4.12, CON4.15, CON4.16, CON4.3, CON4.4, CON4.7, CON4.8
- net RESET: no longer CON4.22
- net TCKOUT: no longer CON4.28
- net TDI: no longer CON4.24
- net TDO: no longer CON4.26
- net TMS: no longer CON4.30
- net 1PPS: now reaches U3.8 (D[9])
- net 1PPS: now also CON4.52
- net +5V_D: now reaches CON4.13
- net +5V_D: now also CON4.14, J4.1
- new net +12V_A: CON4.1, CON4.2
- new net +12V_B: CON4.3, CON4.4
- new net +5V_A: CON4.7, CON4.8, J1.1
- new net +5V_B: CON4.10, CON4.9, J2.1
- new net +5V_C: CON4.11, CON4.12, J3.1
- new net +5V_E: CON4.15, CON4.16, J5.1
Other:
- note removed: "voltage regulator???"
- moved on the sheet: C18, C19, C20, CON4

Commit message: update
Parts:
- C12, C13, C14, C15, C16, C6, C7, C8, C9: value ? -> 100nF
Connections:
- net CAN_H: now also CON4.48; no longer CON4.24
- net CAN_L: now also CON4.44; no longer CON4.20
- net GND: now also CON4.45, CON4.46, CON4.49, CON4.50
Changed lines of the file:
@@
 P 5000 1000
 F 0 "C9" V 5050 1100 50  0000 C CNN
-F 1 "?" V 4900 950 50  0000 C CNN
+F 1 "100nF" V 4925 875 50  0000 C CNN
 F 2 "Capacitors_SMD:C_0603" H 5000 1000 50  0001 C CNN
 F 3 "" H 5000 1000 50  0001 C CNN
@@
 P 5150 1000
 F 0 "C12" V 5200 1125 50  0000 C CNN
-F 1 "?" V 5050 950 50  0000 C CNN
+F 1 "100nF" V 5075 875 50  0000 C CNN
 F 2 "Capacitors_SMD:C_0603" H 5150 1000 50  0001 C CNN
 F 3 "" H 5150 1000 50  0001 C CNN
@@
 P 5300 1000
 F 0 "C13" V 5350 1125 50  0000 C CNN
-F 1 "?" V 5200 950 50  0000 C CNN
+F 1 "100nF" V 5225 875 50  0000 C CNN
 F 2 "Capacitors_SMD:C_0603" H 5300 1000 50  0001 C CNN
 F 3 "" H 5300 1000 50  0001 C CNN
@@
 P 5450 1000
 F 0 "C14" V 5500 1125 50  0000 C CNN
-F 1 "?" V 5350 950 50  0000 C CNN
+F 1 "100nF" V 5375 875 50  0000 C CNN
 F 2 "Capacitors_SMD:C_0603" H 5450 1000 50  0001 C CNN
 F 3 "" H 5450 1000 50  0001 C CNN
@@
 P 5600 1000
 F 0 "C15" V 5650 1125 50  0000 C CNN
-F 1 "?" V 5500 950 50  0000 C CNN
+F 1 "100nF" V 5525 875 50  0000 C CNN
 F 2 "Capacitors_SMD:C_0603" H 5600 1000 50  0001 C CNN
 F 3 "" H 5600 1000 50  0001 C CNN
@@
 P 5750 1000
 F 0 "C16" V 5800 1125 50  0000 C CNN
-F 1 "?" V 5650 950 50  0000 C CNN
+F 1 "100nF" V 5675 875 50  0000 C CNN
 F 2 "Capacitors_SMD:C_0603" H 5750 1000 50  0001 C CNN
 F 3 "" H 5750 1000 50  0001 C CNN
@@
 P 5000 1100
 F 0 "#PWR0103" H 5000 850 50  0001 C CNN
-F 1 "GND" H 5005 927 50  0000 C CNN
+F 1 "GND" H 5000 925 50  0000 C CNN
 F 2 "" H 5000 1100 50  0001 C CNN
 F 3 "" H 5000 1100 50  0001 C CNN
@@
 P 4650 1000
 F 0 "C8" V 4700 1100 50  0000 C CNN
-F 1 "?" V 4550 950 50  0000 C CNN
+F 1 "100nF" V 4750 850 50  0000 C CNN
 F 2 "Capacitors_SMD:C_0603" H 4650 1000 50  0001 C CNN
 F 3 "" H 4650 1000 50  0001 C CNN
@@
 P 4500 1000
 F 0 "C7" V 4550 1100 50  0000 C CNN
-F 1 "?" V 4400 950 50  0000 C CNN
+F 1 "100nF" V 4575 850 50  0000 C CNN
 F 2 "Capacitors_SMD:C_0603" H 4500 1000 50  0001 C CNN
 F 3 "" H 4500 1000 50  0001 C CNN
@@
 P 4350 1000
 F 0 "C6" V 4400 1100 50  0000 C CNN
-F 1 "?" V 4250 950 50  0000 C CNN
+F 1 "100nF" V 4425 850 50  0000 C CNN
 F 2 "Capacitors_SMD:C_0603" H 4350 1000 50  0001 C CNN
 F 3 "" H 4350 1000 50  0001 C CNN
@@
 P 4350 1100
 F 0 "#PWR0111" H 4350 850 50  0001 C CNN
-F 1 "GND" H 4355 927 50  0000 C CNN
+F 1 "GND" H 4325 900 50  0000 C CNN
 F 2 "" H 4350 1100 50  0001 C CNN
 F 3 "" H 4350 1100 50  0001 C CNN
@@
 P 4500 1100
 F 0 "#PWR0112" H 4500 850 50  0001 C CNN
-F 1 "GND" H 4505 927 50  0000 C CNN
+F 1 "GND" H 4500 900 50  0000 C CNN
 F 2 "" H 4500 1100 50  0001 C CNN
 F 3 "" H 4500 1100 50  0001 C CNN
@@
 P 4650 1100
 F 0 "#PWR0113" H 4650 850 50  0001 C CNN
-F 1 "GND" H 4655 927 50  0000 C CNN
+F 1 "GND" H 4650 900 50  0000 C CNN
 F 2 "" H 4650 1100 50  0001 C CNN
 F 3 "" H 4650 1100 50  0001 C CNN
@@
 	1    0    0    -1
 $EndComp
-Text GLabel 1700 4000 2    50   BiDi ~ 0
+Text GLabel 1700 5200 2    50   BiDi ~ 0
 CAN_H
-Text GLabel 1700 3800 2    50   BiDi ~ 0
+Text GLabel 1700 5000 2    50   BiDi ~ 0
 CAN_L
 $Comp
@@
 	1050 3900 1100 3900
 Connection ~ 1100 3900
-Wire Wire Line
-	1700 3800 1600 3800
-Wire Wire Line
-	1700 4000 1600 4000
 Text GLabel 1500 5850 0    50   Input ~ 0
 +5V_A
@@
 Wire Wire Line
 	4050 3500 3650 3500
+$Comp
+L power:GND #PWR?
+U 1 1 5B461461
+P 1025 5300
+F 0 "#PWR?" H 1025 5050 50  0001 C CNN
+F 1 "GND" H 1030 5127 50  0000 C CNN
+F 2 "" H 1025 5300 50  0001 C CNN
+F 3 "" H 1025 5300 50  0001 C CNN
+	1    1025 5300
+	0    1    1    0
+$EndComp
+Wire Wire Line
+	1600 5300 1100 5300
+Wire Wire Line
+	1025 5300 1100 5300
+Connection ~ 1100 5300
+Wire Wire Line
+	1700 5200 1600 5200
+Wire Wire Line
+	1600 5100 1100 5100
+$Comp
+L power:GND #PWR?
+U 1 1 5B4ADB17
+P 1025 5100
+F 0 "#PWR?" H 1025 4850 50  0001 C CNN
+F 1 "GND" H 1030 4927 50  0000 C CNN
+F 2 "" H 1025 5100 50  0001 C CNN
+F 3 "" H 1025 5100 50  0001 C CNN
+	1    1025 5100
+	0    1    1    0
+$EndComp
+Wire Wire Line
+	1025 5100 1100 5100
+Connection ~ 1100 5100
+Wire Wire Line
+	1700 5000 1600 5000
 Wire Bus Line
 	7900 2600 7900 4300

Commit message: update
Parts:
- CON1, CON2: symbol Connector:Conn_Coaxial -> TRX_MODULE-rescue:Conn_Coaxial-Connector
- U4: symbol interface:MCP2561-E-SN -> TRX_MODULE-rescue:MCP2561-E-SN-interface
Changed lines of the file:
@@
 $EndComp
 $Comp
-L Connector:Conn_Coaxial CON1
+L TRX_MODULE-rescue:Conn_Coaxial-Connector CON1
 U 1 1 5B00761C
 P 10400 2100
@@
 $EndComp
 $Comp
-L Connector:Conn_Coaxial CON2
+L TRX_MODULE-rescue:Conn_Coaxial-Connector CON2
 U 1 1 5B01E849
 P 10400 3800
@@
 CAN_RX
 $Comp
-L interface:MCP2561-E-SN U4
+L TRX_MODULE-rescue:MCP2561-E-SN-interface U4
 U 1 1 5B2E06B6
 P 2375 2200
